Commit message: Correction du dossier gripper et ajout des fichiers

File: src/ur_sim/urdf/ur3e_gripper.urdf.xacro (robot description, xacro)
@@ -131,5 +131,5 @@
     <origin xyz="0 0 0" rpy="0 0 0"/>
   </joint>
-  <ros2_control name="OnRobotGripper" type="system">
+<ros2_control name="OnRobotGripper" type="system">
     <hardware>
       <plugin>gz_ros2_control/GazeboSimSystem</plugin>
@@ -137,5 +137,14 @@
     <joint name="left_finger_joint">
       <command_interface name="position"/>
-      <state_interface name="position"/>
+      <state_interface name="position">
+        <param name="initial_value">0.0</param>
+      </state_interface>
+      <state_interface name="velocity"/>
+    </joint>
+    <joint name="right_finger_joint">
+      <command_interface name="position"/>
+      <state_interface name="position">
+        <param name="initial_value">0.0</param>
+      </state_interface>
       <state_interface name="velocity"/>
     </joint>
